File: board/board.kicad_pcb (KiCad board)
At the start: 2 copper layers, 21 x 13 mm, 1 part

Commit message: initial
Parts:
- added C1: 100pF, Capacitor_SMD:C_0402_1005Metric, F.Cu at (149.2, 91.9)
- added J1: 008_USB, on_edge:on_edge_2x05_host, F.Cu at (161.0, 96.5)
- added J2: USB4105-GF-A, b051:GCT_USB4105-GF-A, F.Cu at (142.6, 96.2)
- added R1: 0R, Resistor_SMD:R_0603_1608Metric, F.Cu at (154.3, 94.5)
- added R2: d.n.p, Resistor_SMD:R_0603_1608Metric, F.Cu at (154.2, 100.5)
- added R3: 5.1k, Resistor_SMD:R_0402_1005Metric, F.Cu at (149.3, 95.0)
- added R4: 5.1k, Resistor_SMD:R_0402_1005Metric, F.Cu at (149.7, 97.9)
- LOGO1: moved to B.Cu
- moved LOGO1 1.92 mm to (151.8, 99.8), turned to 180 degrees
Routing:
- net GND: track 0.00 -> 22.5 mm
- net /usb-c/VBUS: track 0.00 -> 20.9 mm, vias 0 -> 3
- net Net-(J2-PadG1): track 0.00 -> 18.9 mm
- net /usb-c/DM: track 0.00 -> 14.5 mm, vias 0 -> 2
- net /usb-c/DP: track 0.00 -> 14.0 mm, vias 0 -> 2
- net Net-(J1-Pad2): track 0.00 -> 3.53 mm
- net Net-(J1-Pad10): track 0.00 -> 3.45 mm, vias 0 -> 1
- net Net-(J2-PadB5): track 0.00 -> 1.93 mm
- net Net-(J2-PadA5): track 0.00 -> 1.45 mm
Other:
- outline, holes or cut-outs redrawn
- board text added: "osf.008"
- board text added: "osf.b051.v1.0"
